Commit message: point cloud is working, calibration hand eye;

File: franka_description/robots/panda_arm_hand.urdf.xacro (robot description, xacro)
@@ -3,5 +3,9 @@
   <xacro:include filename="$(find franka_description)/robots/panda_arm.xacro"/>
   <xacro:include filename="$(find franka_description)/robots/hand.xacro"/>
+  <xacro:include filename="$(find ros_sensors)/urdf/intel_d435.urdf.xacro"/>
   <xacro:panda_arm />
   <xacro:hand ns="panda" rpy="0 0 ${-pi/4}" connected_to="panda_link8"/>
+  <xacro:sensor_r430 prefix="" prefix_topic="" parent="panda_link8">
+    <origin xyz="0.06 -0.06 0.025" rpy="${pi} ${-pi/2} ${-pi/4}" />
+  </xacro:sensor_r430>
 </robot>

Commit message: automated 3d data collection

File: franka_description/robots/panda_arm_hand.urdf.xacro (robot description, xacro)
@@ -9,3 +9,15 @@
     <origin xyz="0.06 -0.06 0.025" rpy="${pi} ${-pi/2} ${-pi/4}" />
   </xacro:sensor_r430>
+  <!-- <link name="xela_sensor_frame"/> -->
+  <!-- <joint name="xela_sensor_joint" type="fixed">
+    <parent link="panda_leftfinger"/>
+    <child link="xela_sensor_frame"/>
+    <origin xyz="0.025 0.01 0.065 " rpy="0 0 0"/>
+  </joint> -->
+  <link name="xela_sensor_frame"/>
+  <joint name="xela_sensor_joint" type="fixed">
+    <parent link="panda_link8"/>
+    <child link="xela_sensor_frame"/>
+    <origin xyz="0.025 -0.011 0.123" rpy="0 0 0"/>
+  </joint>
 </robot>

File: panda_moveit_config/config/panda_arm.xacro (robot description, xacro)
@@ -66,4 +66,24 @@
       <joint name="panda_joint6" value="2.6326718765970223" />
       <joint name="panda_joint7" value="0.33089223800978584" />
+    </group_state>
+<!-- [-0.013777106709055475, 0.39804385980602447, 0.07457416601831604, -2.1136673020640075, -0.01011319098046733, 2.4297943443565524, 1.4367238919482461, -->
+    <group_state name="nippleC" group="panda_arm">
+      <joint name="panda_joint1" value="-0.013777106709055475" />
+      <joint name="panda_joint2" value="0.39804385980602447" />
+      <joint name="panda_joint3" value="0.07457416601831604" />
+      <joint name="panda_joint4" value="-2.1136673020640075" />
+      <joint name="panda_joint5" value="-0.01011319098046733" />
+      <joint name="panda_joint6" value="2.4297943443565524" />
+      <joint name="panda_joint7" value="1.4367238919482461" />
+    </group_state>
+<!-- [0.0033272228759615727, 0.17591706981655317, 0.0461060038543639, -2.480672533383676, -0.005410064732307921, 2.602337698035745, 0.852062157835232, -->
+    <group_state name="nippleD" group="panda_arm">
+      <joint name="panda_joint1" value="0.0033272228759615727" />
+      <joint name="panda_joint2" value="0.17591706981655317" />
+      <joint name="panda_joint3" value="0.0461060038543639" />
+      <joint name="panda_joint4" value="-2.480672533383676" />
+      <joint name="panda_joint5" value="-0.005410064732307921" />
+      <joint name="panda_joint6" value="2.602337698035745" />
+      <joint name="panda_joint7" value="0.852062157835232" />
     </group_state>
     <!-- <group_state name="poseA" group="panda_arm">

File: panda_moveit_config/config/panda_arm_hand.srdf.xacro (robot description, xacro)
@@ -1,46 +1,151 @@
-<?xml version='1.0' encoding='utf-8'?>
+<?xml version="1.0" ?>
 <!--This does not replace URDF, and is not an extension of URDF.
     This is a format for representing semantic information about the robot structure.
     A URDF file must exist for this robot as well, where the joints and the links that are referenced are defined
 -->
-<robot xmlns:xacro="http://www.ros.org/wiki/xacro" name="panda">
-  <xacro:include filename="$(find panda_moveit_config)/config/panda_arm.xacro" />
-  <xacro:include filename="$(find panda_moveit_config)/config/hand.xacro" />
-  <xacro:panda_arm />
-  <xacro:hand />
-  <!--GROUPS: Representation of a set of joints and links. This can be useful for specifying DOF to plan for, defining arms, end effectors, etc-->
-  <!--LINKS: When a link is specified, the parent joint of that link (if it exists) is automatically included-->
-  <!--JOINTS: When a joint is specified, the child link of that joint (which will always exist) is automatically included-->
-  <!--CHAINS: When a chain is specified, all the links along the chain (including endpoints) are included in the group. Additionally, all the joints that are parents to included links are also included. This means that joints along the chain and the parent joint of the base link are included in the group-->
-  <!--SUBGROUPS: Groups can also be formed by referencing to already defined group names-->
-  <group name="panda_arm_hand">
-    <group name="panda_arm" />
-    <group name="hand" />
-  </group>
-  <!--GROUP STATES: Purpose: Define a named state for a particular group, in terms of joint values. This is useful to define states like 'folded arms'-->
-  <group_state name="ready" group="panda_arm_hand">
-    <joint name="panda_joint1" value="0" />
-    <joint name="panda_joint2" value="-0.785" />
-    <joint name="panda_joint3" value="0" />
-    <joint name="panda_joint4" value="-2.356" />
-    <joint name="panda_joint5" value="0" />
-    <joint name="panda_joint6" value="1.571" />
-    <joint name="panda_joint7" value="0.785" />
-  </group_state>
-  <!--END EFFECTOR: Purpose: Represent information about an end effector.-->
-  <end_effector name="hand" parent_link="panda_hand" group="hand" parent_group="panda_arm_hand" />
-  <!--DISABLE COLLISIONS: By default it is assumed that any link of the robot could potentially come into collision with any other link in the robot. This tag disables collision checking between a specified pair of links. -->
-  <disable_collisions link1="panda_hand" link2="panda_link3" reason="Never" />
-  <disable_collisions link1="panda_hand" link2="panda_link4" reason="Never" />
-  <disable_collisions link1="panda_hand" link2="panda_link5" reason="Default" />
-  <disable_collisions link1="panda_hand" link2="panda_link6" reason="Never" />
-  <disable_collisions link1="panda_hand" link2="panda_link7" reason="Adjacent" />
-  <disable_collisions link1="panda_leftfinger" link2="panda_link3" reason="Never" />
-  <disable_collisions link1="panda_leftfinger" link2="panda_link4" reason="Never" />
-  <disable_collisions link1="panda_leftfinger" link2="panda_link6" reason="Never" />
-  <disable_collisions link1="panda_leftfinger" link2="panda_link7" reason="Never" />
-  <disable_collisions link1="panda_link3" link2="panda_rightfinger" reason="Never" />
-  <disable_collisions link1="panda_link4" link2="panda_rightfinger" reason="Never" />
-  <disable_collisions link1="panda_link6" link2="panda_rightfinger" reason="Never" />
-  <disable_collisions link1="panda_link7" link2="panda_rightfinger" reason="Never" />
+<robot name="panda">
+    <!--GROUPS: Representation of a set of joints and links. This can be useful for specifying DOF to plan for, defining arms, end effectors, etc-->
+    <!--LINKS: When a link is specified, the parent joint of that link (if it exists) is automatically included-->
+    <!--JOINTS: When a joint is specified, the child link of that joint (which will always exist) is automatically included-->
+    <!--CHAINS: When a chain is specified, all the links along the chain (including endpoints) are included in the group. Additionally, all the joints that are parents to included links are also included. This means that joints along the chain and the parent joint of the base link are included in the group-->
+    <!--SUBGROUPS: Groups can also be formed by referencing to already defined group names-->
+    <group name="panda_arm">
+        <link name="panda_link0" />
+        <link name="panda_link1" />
+        <link name="panda_link2" />
+        <link name="panda_link3" />
+        <link name="panda_link4" />
+        <link name="panda_link5" />
+        <link name="panda_link6" />
+        <link name="panda_link7" />
+        <link name="panda_link8" />
+        <joint name="panda_joint1" />
+        <joint name="panda_joint2" />
+        <joint name="panda_joint3" />
+        <joint name="panda_joint4" />
+        <joint name="panda_joint5" />
+        <joint name="panda_joint6" />
+        <joint name="panda_joint7" />
+        <joint name="panda_joint8" />
+        <chain base_link="panda_link0" tip_link="xela_sensor_frame" />
+    </group>
+    <group name="hand">
+        <link name="panda_hand" />
+        <link name="panda_leftfinger" />
+        <link name="panda_rightfinger" />
+        <joint name="panda_finger_joint1" />
+    </group>
+    <group name="panda_arm_hand">
+        <group name="panda_arm" />
+        <group name="hand" />
+    </group>
+    <!--GROUP STATES: Purpose: Define a named state for a particular group, in terms of joint values. This is useful to define states like 'folded arms'-->
+    <group_state name="ready" group="panda_arm">
+        <joint name="panda_joint1" value="0" />
+        <joint name="panda_joint2" value="-0.785" />
+        <joint name="panda_joint3" value="0" />
+        <joint name="panda_joint4" value="-2.356" />
+        <joint name="panda_joint5" value="0" />
+        <joint name="panda_joint6" value="1.571" />
+        <joint name="panda_joint7" value="0.785" />
+    </group_state>
+    <group_state name="poseA" group="panda_arm">
+        <joint name="panda_joint1" value="0" />
+        <joint name="panda_joint2" value="-0.242787" />
+        <joint name="panda_joint3" value="-0.0192369" />
+        <joint name="panda_joint4" value="-1.87651" />
+        <joint name="panda_joint5" value="-0.00768018" />
+        <joint name="panda_joint6" value="1.57473" />
+        <joint name="panda_joint7" value="0.813186" />
+    </group_state>
+    <group_state name="nippleA" group="panda_arm">
+        <joint name="panda_joint1" value="-0.0543767" />
+        <joint name="panda_joint2" value="0.471072" />
+        <joint name="panda_joint3" value="0.171324" />
+        <joint name="panda_joint4" value="-2.03379" />
+        <joint name="panda_joint5" value="-0.0378312" />
+        <joint name="panda_joint6" value="2.4434" />
+        <joint name="panda_joint7" value="0.951624" />
+    </group_state>
+    <group_state name="nippleB" group="panda_arm">
+        <joint name="panda_joint1" value="-0.0507545" />
+        <joint name="panda_joint2" value="0.336191" />
+        <joint name="panda_joint3" value="0.240567" />
+        <joint name="panda_joint4" value="-2.26739" />
+        <joint name="panda_joint5" value="-0.149971" />
+        <joint name="panda_joint6" value="2.63267" />
+        <joint name="panda_joint7" value="0.330892" />
+    </group_state>
+    <group_state name="nippleC" group="panda_arm">
+        <joint name="panda_joint1" value="-0.0137771" />
+        <joint name="panda_joint2" value="0.398044" />
+        <joint name="panda_joint3" value="0.0745742" />
+        <joint name="panda_joint4" value="-2.11367" />
+        <joint name="panda_joint5" value="-0.0101132" />
+        <joint name="panda_joint6" value="2.42979" />
+        <joint name="panda_joint7" value="1.43672" />
+    </group_state>
+    <group_state name="nippleD" group="panda_arm">
+        <joint name="panda_joint1" value="0.00332722" />
+        <joint name="panda_joint2" value="0.175917" />
+        <joint name="panda_joint3" value="0.046106" />
+        <joint name="panda_joint4" value="-2.48067" />
+        <joint name="panda_joint5" value="-0.00541006" />
+        <joint name="panda_joint6" value="2.60234" />
+        <joint name="panda_joint7" value="0.852062" />
+    </group_state>
+    <group_state name="ready" group="panda_arm_hand">
+        <joint name="panda_joint1" value="0" />
+        <joint name="panda_joint2" value="-0.785" />
+        <joint name="panda_joint3" value="0" />
+        <joint name="panda_joint4" value="-2.356" />
+        <joint name="panda_joint5" value="0" />
+        <joint name="panda_joint6" value="1.571" />
+        <joint name="panda_joint7" value="0.785" />
+    </group_state>
+    <!--END EFFECTOR: Purpose: Represent information about an end effector.-->
+    <end_effector name="hand" parent_link="panda_hand" group="hand" parent_group="panda_arm_hand" />
+    <!--DISABLE COLLISIONS: By default it is assumed that any link of the robot could potentially come into collision with any other link in the robot. This tag disables collision checking between a specified pair of links. -->
+    <disable_collisions link1="_camera_link" link2="panda_hand" reason="Adjacent" />
+    <disable_collisions link1="_camera_link" link2="panda_leftfinger" reason="Never" />
+    <disable_collisions link1="_camera_link" link2="panda_link3" reason="Never" />
+    <disable_collisions link1="_camera_link" link2="panda_link4" reason="Never" />
+    <disable_collisions link1="_camera_link" link2="panda_link6" reason="Never" />
+    <disable_collisions link1="_camera_link" link2="panda_link7" reason="Adjacent" />
+    <disable_collisions link1="_camera_link" link2="panda_rightfinger" reason="Never" />
+    <disable_collisions link1="panda_hand" link2="panda_leftfinger" reason="Adjacent" />
+    <disable_collisions link1="panda_hand" link2="panda_link3" reason="Never" />
+    <disable_collisions link1="panda_hand" link2="panda_link4" reason="Never" />
+    <disable_collisions link1="panda_hand" link2="panda_link5" reason="Default" />
+    <disable_collisions link1="panda_hand" link2="panda_link6" reason="Never" />
+    <disable_collisions link1="panda_hand" link2="panda_link7" reason="Adjacent" />
+    <disable_collisions link1="panda_hand" link2="panda_rightfinger" reason="Adjacent" />
+    <disable_collisions link1="panda_leftfinger" link2="panda_link3" reason="Never" />
+    <disable_collisions link1="panda_leftfinger" link2="panda_link4" reason="Never" />
+    <disable_collisions link1="panda_leftfinger" link2="panda_link6" reason="Never" />
+    <disable_collisions link1="panda_leftfinger" link2="panda_link7" reason="Never" />
+    <disable_collisions link1="panda_leftfinger" link2="panda_rightfinger" reason="Default" />
+    <disable_collisions link1="panda_link0" link2="panda_link1" reason="Adjacent" />
+    <disable_collisions link1="panda_link0" link2="panda_link2" reason="Never" />
+    <disable_collisions link1="panda_link0" link2="panda_link3" reason="Never" />
+    <disable_collisions link1="panda_link0" link2="panda_link4" reason="Never" />
+    <disable_collisions link1="panda_link1" link2="panda_link2" reason="Adjacent" />
+    <disable_collisions link1="panda_link1" link2="panda_link3" reason="Never" />
+    <disable_collisions link1="panda_link1" link2="panda_link4" reason="Never" />
+    <disable_collisions link1="panda_link2" link2="panda_link3" reason="Adjacent" />
+    <disable_collisions link1="panda_link2" link2="panda_link4" reason="Never" />
+    <disable_collisions link1="panda_link3" link2="panda_link4" reason="Adjacent" />
+    <disable_collisions link1="panda_link3" link2="panda_link5" reason="Never" />
+    <disable_collisions link1="panda_link3" link2="panda_link6" reason="Never" />
+    <disable_collisions link1="panda_link3" link2="panda_link7" reason="Never" />
+    <disable_collisions link1="panda_link3" link2="panda_rightfinger" reason="Never" />
+    <disable_collisions link1="panda_link4" link2="panda_link5" reason="Adjacent" />
+    <disable_collisions link1="panda_link4" link2="panda_link6" reason="Never" />
+    <disable_collisions link1="panda_link4" link2="panda_link7" reason="Never" />
+    <disable_collisions link1="panda_link4" link2="panda_rightfinger" reason="Never" />
+    <disable_collisions link1="panda_link5" link2="panda_link6" reason="Adjacent" />
+    <disable_collisions link1="panda_link5" link2="panda_link7" reason="Default" />
+    <disable_collisions link1="panda_link6" link2="panda_link7" reason="Adjacent" />
+    <disable_collisions link1="panda_link6" link2="panda_rightfinger" reason="Never" />
+    <disable_collisions link1="panda_link7" link2="panda_rightfinger" reason="Never" />
 </robot>

Commit message: validaing palpation results

File: franka_description/robots/panda_arm_hand.urdf.xacro (robot description, xacro)
@@ -6,4 +6,7 @@
   <xacro:panda_arm />
   <xacro:hand ns="panda" rpy="0 0 ${-pi/4}" connected_to="panda_link8"/>
+  <!-- <xacro:sensor_r430 prefix="" prefix_topic="" parent="panda_link8">
+    <origin xyz="0.06 -0.06 0.025" rpy="${pi} ${-pi/2} ${-pi/4}" />
+  </xacro:sensor_r430> -->
   <xacro:sensor_r430 prefix="" prefix_topic="" parent="panda_link8">
     <origin xyz="0.06 -0.06 0.025" rpy="${pi} ${-pi/2} ${-pi/4}" />

Commit message: complete success

File: franka_description/robots/panda_arm_hand.urdf.xacro (robot description, xacro)
@@ -9,6 +9,9 @@
     <origin xyz="0.06 -0.06 0.025" rpy="${pi} ${-pi/2} ${-pi/4}" />
   </xacro:sensor_r430> -->
+  <!-- <xacro:sensor_r430 prefix="" prefix_topic="" parent="panda_link8">
+    <origin xyz="0.06 -0.06 0.025" rpy="${pi} ${-pi/2} ${-pi/4}" />
+  </xacro:sensor_r430> -->
   <xacro:sensor_r430 prefix="" prefix_topic="" parent="panda_link8">
-    <origin xyz="0.06 -0.06 0.025" rpy="${pi} ${-pi/2} ${-pi/4}" />
+    <origin xyz="0.06 -0.06 0.0325" rpy="${pi} ${-pi/2} ${-pi/4}" />
   </xacro:sensor_r430>
   <!-- <link name="xela_sensor_frame"/> -->
